Commit message: Gazebo launch.py

File: brobot_ws/src/brobot_description/urdf/brobot.urdf (robot description, URDF)
Before this commit: robot brobot, 3 links, 2 joints
Links:
- link base_link: mass None -> 0.25; geometry collision cylinder length=0.11 radius=0.045; visual cylinder length=0.11 radius=0.045
- link left_wheel: mass None -> 0.03; geometry collision cylinder length=0.015 radius=0.025; visual cylinder length=0.015 radius=0.025
- link right_wheel: mass None -> 0.03; geometry collision cylinder length=0.015 radius=0.025; visual cylinder length=0.015 radius=0.025
Joints:
- joint left_wheel_joint: origin xyz=0 0.06 -0.03 rpy=1.5708 0 0 -> xyz=0 0.05 -0.03 rpy=1.5708 0 0; type fixed -> continuous
- joint right_wheel_joint: origin xyz=0 -0.06 -0.03 rpy=1.5708 0 0 -> xyz=0 -0.05 -0.03 rpy=1.5708 0 0

Commit message: Update brobot.urdf

File: brobot_ws/src/brobot_description/urdf/brobot.urdf (robot description, URDF)
Before this commit: robot brobot, 3 links, 2 joints
Joints:
- joint left_wheel_joint: axis (none) -> 0 0 1
- joint right_wheel_joint: axis (none) -> 0 0 1; type fixed -> continuous
