Commit message: Added Gazebo Launch

File: deskbot_ws/src/deskbot_description/urdf/deskbot.urdf (robot description, URDF)
Before this commit: robot deskbot, 5 links, 4 joints
Links:
- added link left_len, mass 1.0; visual cylinder length=0.05 radius=0.05
- added link left_pupil, mass 1.0; visual cylinder length=0.05 radius=0.035
- added link right_len, mass 1.0; visual cylinder length=0.05 radius=0.05
- added link right_pupil, mass 1.0; visual cylinder length=0.05 radius=0.035
- link back_left_wheel: mass None -> 1.0
- link back_right_wheel: mass None -> 1.0
- link base_link: mass None -> 1.0
- link front_left_wheel: mass None -> 1.0
- link front_right_wheel: mass None -> 1.0
Joints:
- added joint left_len_joint: type fixed, parent base_link, child left_len, origin xyz=0.35 0.15 0.02
- added joint left_pupil_joint: type fixed, parent base_link, child left_pupil, origin xyz=0.355 0.15 0.02
- added joint right_len_joint: type fixed, parent base_link, child right_len, origin xyz=0.35 -0.15 0.02
- added joint right_pupil_joint: type fixed, parent base_link, child right_pupil, origin xyz=0.355 -0.15 0.02
- joint back_left_wheel_joint: origin xyz=-0.15 0.30 -0.15 -> xyz=-0.20 0.30 -0.15
- joint back_right_wheel_joint: origin xyz=-0.15 -0.30 -0.15 -> xyz=-0.20 -0.30 -0.15
- joint front_left_wheel_joint: origin xyz=0.15 0.30 -0.15 -> xyz=0.20 0.30 -0.15
- joint front_right_wheel_joint: origin xyz=0.15 -0.30 -0.15 -> xyz=0.20 -0.30 -0.15

Commit message: Added collision to deskbot's urdf

File: deskbot_ws/src/deskbot_description/urdf/deskbot.urdf (robot description, URDF)
Before this commit: robot deskbot, 9 links, 8 joints
Links:
- link back_left_wheel: geometry collision cylinder length=0.1 radius=0.15; visual cylinder length=0.1 radius=0.15
- link back_right_wheel: geometry collision cylinder length=0.1 radius=0.15; visual cylinder length=0.1 radius=0.15
- link base_link: geometry collision box size=0.7 0.5 0.3; visual box size=0.7 0.5 0.3
- link front_left_wheel: geometry collision cylinder length=0.1 radius=0.15; visual cylinder length=0.1 radius=0.15
- link front_right_wheel: geometry collision cylinder length=0.1 radius=0.15; visual cylinder length=0.1 radius=0.15

Commit message: Working on Battery and Led Panel nodes

File: deskbot_ws/src/deskbot_description/urdf/deskbot.urdf (robot description, URDF)
Before this commit: robot deskbot, 9 links, 8 joints
Links:
- link base_link: mass 1.0 -> 5.0
- link left_len: mass 1.0 -> 0.01
- link left_pupil: mass 1.0 -> 0.01
- link right_len: mass 1.0 -> 0.01
- link right_pupil: mass 1.0 -> 0.01

Commit message: Added Gazebo simulation world with desk

File: deskbot_ws/src/deskbot_description/urdf/deskbot.urdf (robot description, URDF)
Before this commit: robot deskbot, 9 links, 8 joints
Links:
- link back_left_wheel: mass 1.0 -> 0.05; geometry collision cylinder length=0.02 radius=0.03; visual cylinder length=0.02 radius=0.03
- link back_right_wheel: mass 1.0 -> 0.05; geometry collision cylinder length=0.02 radius=0.03; visual cylinder length=0.02 radius=0.03
- link base_link: mass 5.0 -> 0.4; geometry collision box size=0.14 0.10 0.06; visual box size=0.14 0.10 0.06
- link front_left_wheel: mass 1.0 -> 0.05; geometry collision cylinder length=0.02 radius=0.03; visual cylinder length=0.02 radius=0.03
- link front_right_wheel: mass 1.0 -> 0.05; geometry collision cylinder length=0.02 radius=0.03; visual cylinder length=0.02 radius=0.03
- link left_len: mass 0.01 -> 0.001; geometry visual cylinder length=0.01 radius=0.01
- link left_pupil: mass 0.01 -> 0.001; geometry visual cylinder length=0.01 radius=0.007
- link right_len: mass 0.01 -> 0.001; geometry visual cylinder length=0.01 radius=0.01
- link right_pupil: mass 0.01 -> 0.001; geometry visual cylinder length=0.01 radius=0.007
Joints:
- joint back_left_wheel_joint: origin xyz=-0.20 0.30 -0.15 -> xyz=-0.04 0.065 -0.02
- joint back_right_wheel_joint: origin xyz=-0.20 -0.30 -0.15 -> xyz=-0.04 -0.065 -0.02
- joint front_left_wheel_joint: origin xyz=0.20 0.30 -0.15 -> xyz=0.04 0.065 -0.02
- joint front_right_wheel_joint: origin xyz=0.20 -0.30 -0.15 -> xyz=0.04 -0.065 -0.02
- joint left_len_joint: origin xyz=0.35 0.15 0.02 -> xyz=0.07 0.03 0.005
- joint left_pupil_joint: origin xyz=0.355 0.15 0.02 -> xyz=0.071 0.03 0.005
- joint right_len_joint: origin xyz=0.35 -0.15 0.02 -> xyz=0.07 -0.03 0.005
- joint right_pupil_joint: origin xyz=0.355 -0.15 0.02 -> xyz=0.071 -0.03 0.005
